File: Pro/PCB/Lily58_Pro.kicad_sch (KiCad schematic)
At the start: 83 parts, among them J1 LED, J2 4PIN, J3 OLED, P1 i2c_pin, P2 i2c_pin, SW1 SW_PUSH, SW10 SW_PUSH, SW11 SW_PUSH, SW12 SW_PUSH, SW13 SW_PUSH, SW14 SW_PUSH, SW15 SW_PUSH, SW16 SW_PUSH, SW17 SW_PUSH, SW18 SW_PUSH, SW19 SW_PUSH, SW2 SW_PUSH, SW20 SW_PUSH, SW21 SW_PUSH, SW22 SW_PUSH, SW23 SW_PUSH, SW24 SW_PUSH, SW25 SW_PUSH, SW26 SW_PUSH, SW27 SW_PUSH, SW28 SW_PUSH, SW29 SW_PUSH, SW3 SW_PUSH, SW4 SW_PUSH, SW5 SW_PUSH, SW6 SW_PUSH, SW7 SW_PUSH, SW8 SW_PUSH, SW9 SW_PUSH, U1 ProMicro

Commit message: Update project according KiCAD 7
Parts:
- D1, D10, D11, D12, D13, D14, D15, D16, D17, D18, D19, D2, D20, D21, D22, D23, D24, D25, D26, D27, D28, D29, D3, D4, D5, D6, D7, D8, D9: footprint Lily58-footprint:Diode_SOD123 -> Lily58_Pro:Diode_TH_SOD123
- J1: footprint Lily58-footprint:LED -> Lily58_Pro:LED
- J2: footprint Lily58-footprint:MJ-4PP-9 -> Lily58_Pro:MJ-4PP-9
- J3: footprint Lily58-footprint:OLED_4Pin -> Lily58_Pro:OLED_4Pin
- JP1, JP2, JP3, JP4, JP5, JP6, JP7, JP8: footprint Lily58-footprint:Jumper -> Lily58_Pro:Jumper
- P1, P2: footprint Lily58-footprint:1pin_conn -> Lily58_Pro:1pin_conn
- R1, R2: footprint Lily58-footprint:RESISTOR_mini -> Lily58_Pro:RESISTOR_mini
- RSW1: footprint Lily58-footprint:TACT_SWITCH_TVBP06 -> Lily58_Pro:TACT_SWITCH_TVBP06
- SW1, SW10, SW11, SW12, SW13, SW14, SW15, SW16, SW17, SW18, SW19, SW2, SW20, SW21, SW22, SW23, SW24, SW25, SW26, SW27, SW28, SW29, SW3, SW4, SW5, SW6, SW7, SW8, SW9: footprint Lily58-footprint:CherryMX_KailhLowProfile_Hotswap -> Lily58_Pro:MX_Choc_Hotswap
- TH1, TH2: footprint Lily58-footprint:M2_HOLE_PCB -> Lily58_Pro:HOLE_M2
- TH3, TH4, TH5, TH6, TH7: footprint Lily58-footprint:HOLE_M2_TH -> Lily58_Pro:HOLE_M2_TH
- U1: footprint Lily58-footprint:ProMicro_rev2 -> Lily58_Pro:ProMicro_rev2

Commit message: wireless scheme is almost ready
Parts:
- removed J1: LED, Lily58_Pro:LED, symbol Lily58_Pro-rescue:LED-Lily58-cache
- removed J2: 4PIN, Lily58_Pro:MJ-4PP-9, symbol Lily58_Pro-rescue:MJ-4PP-9-Lily58-cache
- removed P1, P2: i2c_pin, Lily58_Pro:1pin_conn, symbol Lily58_Pro-rescue:i2c_pin-Lily58-cache
- removed R1, R2: R, Lily58_Pro:RESISTOR_mini, symbol Lily58_Pro-rescue:R-Lily58-cache
- removed W1: jumper, Lily58-footprint:jumper_data, symbol Lily58_Pro-rescue:Jumper-Device
- added J1: FS_Battery_Socket, Connector_JST:JST_PH_S2B-PH-K_1x02_P2.00mm_Horizontal, symbol Connector:Conn_01x02_Socket
- added J2: BS_Battery_Socket, Connector_JST:JST_PH_S2B-PH-K_1x02_P2.00mm_Horizontal, symbol Connector:Conn_01x02_Socket
- added JP10, JP11, JP12, JP9: ~, Lily58_Pro:Jumper, symbol Lily58_Pro-rescue:Jumper_NO_Small-Device
- added SW30: FS_SW_SPDT, marbastlib-various:SW_MSK12C02-HB, symbol Switch:SW_SPDT
- added SW31: BS_SW_SPDT, marbastlib-various:SW_MSK12C02-HB, symbol Switch:SW_SPDT
Connections:
- net GND: now also JP11.1, JP9.1
- net RAW: now reaches U1.24 (RAW)
- net RAW: now also SW30.2 (B), SW31.2 (B)
- net LED: no longer names the net of U1.1 (TX(PD3))
- new net: J1.1 (Pin_1), J1.2 (Pin_2), J2.1 (Pin_1), J2.2 (Pin_2), JP10.2, JP11.2, JP12.2, JP9.2
- new net BAT: JP10.1, JP12.1, SW30.3 (C), SW31.3 (C)
- no-connect marks 4 -> 6
Other:
- moved on the sheet: J3, JP1, JP2, JP3, JP4, JP5, JP6, JP7, JP8, RSW1

Commit message: itermediate version
Parts:
- renumbered SW31 to B_Switch1, SW30 to F_Switch1, JP1 to JP_GND1, JP8 to JP_GND2, JP3 to JP_SCL1, JP6 to JP_SCL2, JP4 to JP_SDA1, JP5 to JP_SDA2, JP2 to JP_VCC1, JP7 to JP_VCC2
Other:
- moved on the sheet: JP_GND1, JP_GND2, JP_SCL1, JP_SCL2, JP_SDA1, JP_SDA2, JP_VCC1, JP_VCC2

Commit message: It's done. v0.1 ready to print
Parts:
- D1, D10, D11, D12, D13, D14, D15, D16, D17, D18, D19, D2, D20, D21, D22, D23, D24, D25, D26, D27, D28, D29, D3, D4, D5, D6, D7, D8, D9: footprint Lily58_Pro:Diode_TH_SOD123 -> Hedgehog:Diode_SOD123
Changed lines of the file:
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@@
       (effects (font (size 1.27 1.27)) (justify right))
     )
-    (property "Footprint" "Lily58_Pro:Diode_TH_SOD123" (at 154.94 60.96 0)
+    (property "Footprint" "Hedgehog:Diode_SOD123" (at 154.94 60.96 0)
       (effects (font (size 1.27 1.27)) hide)
     )
@@
       (effects (font (size 1.27 1.27)) (justify right))
     )
-    (property "Footprint" "Lily58_Pro:Diode_TH_SOD123" (at 175.26 60.96 0)
+    (property "Footprint" "Hedgehog:Diode_SOD123" (at 175.26 60.96 0)
       (effects (font (size 1.27 1.27)) hide)
     )
@@
       (effects (font (size 1.27 1.27)) (justify right))
     )
-    (property "Footprint" "Lily58_Pro:Diode_TH_SOD123" (at 195.58 60.96 0)
+    (property "Footprint" "Hedgehog:Diode_SOD123" (at 195.58 60.96 0)
       (effects (font (size 1.27 1.27)) hide)
     )
@@
       (effects (font (size 1.27 1.27)) (justify right))
     )
-    (property "Footprint" "Lily58_Pro:Diode_TH_SOD123" (at 215.9 60.96 0)
+    (property "Footprint" "Hedgehog:Diode_SOD123" (at 215.9 60.96 0)
       (effects (font (size 1.27 1.27)) hide)
     )
@@
       (effects (font (size 1.27 1.27)) (justify right))
     )
-    (property "Footprint" "Lily58_Pro:Diode_TH_SOD123" (at 236.22 60.96 0)
+    (property "Footprint" "Hedgehog:Diode_SOD123" (at 236.22 60.96 0)
       (effects (font (size 1.27 1.27)) hide)
     )
@@
       (effects (font (size 1.27 1.27)) (justify right))
     )
-    (property "Footprint" "Lily58_Pro:Diode_TH_SOD123" (at 256.54 60.96 0)
+    (property "Footprint" "Hedgehog:Diode_SOD123" (at 256.54 60.96 0)
       (effects (font (size 1.27 1.27)) hide)
     )
@@
       (effects (font (size 1.27 1.27)) (justify right))
     )
-    (property "Footprint" "Lily58_Pro:Diode_TH_SOD123" (at 154.94 77.47 0)
+    (property "Footprint" "Hedgehog:Diode_SOD123" (at 154.94 77.47 0)
       (effects (font (size 1.27 1.27)) hide)
     )
@@
       (effects (font (size 1.27 1.27)) (justify right))
     )
-    (property "Footprint" "Lily58_Pro:Diode_TH_SOD123" (at 175.26 77.47 0)
+    (property "Footprint" "Hedgehog:Diode_SOD123" (at 175.26 77.47 0)
       (effects (font (size 1.27 1.27)) hide)
     )
@@
       (effects (font (size 1.27 1.27)) (justify right))
     )
-    (property "Footprint" "Lily58_Pro:Diode_TH_SOD123" (at 195.58 77.47 0)
+    (property "Footprint" "Hedgehog:Diode_SOD123" (at 195.58 77.47 0)
       (effects (font (size 1.27 1.27)) hide)
     )
@@
       (effects (font (size 1.27 1.27)) (justify right))
     )
-    (property "Footprint" "Lily58_Pro:Diode_TH_SOD123" (at 215.9 77.47 0)
+    (property "Footprint" "Hedgehog:Diode_SOD123" (at 215.9 77.47 0)
       (effects (font (size 1.27 1.27)) hide)
     )
@@
       (effects (font (size 1.27 1.27)) (justify right))
     )
-    (property "Footprint" "Lily58_Pro:Diode_TH_SOD123" (at 236.22 77.47 0)
+    (property "Footprint" "Hedgehog:Diode_SOD123" (at 236.22 77.47 0)
       (effects (font (size 1.27 1.27)) hide)
     )
@@
       (effects (font (size 1.27 1.27)) (justify right))
     )
-    (property "Footprint" "Lily58_Pro:Diode_TH_SOD123" (at 256.54 77.47 0)
+    (property "Footprint" "Hedgehog:Diode_SOD123" (at 256.54 77.47 0)
       (effects (font (size 1.27 1.27)) hide)
     )
@@
       (effects (font (size 1.27 1.27)) (justify right))
     )
-    (property "Footprint" "Lily58_Pro:Diode_TH_SOD123" (at 154.94 93.98 0)
+    (property "Footprint" "Hedgehog:Diode_SOD123" (at 154.94 93.98 0)
       (effects (font (size 1.27 1.27)) hide)
     )
@@
       (effects (font (size 1.27 1.27)) (justify right))
     )
-    (property "Footprint" "Lily58_Pro:Diode_TH_SOD123" (at 175.26 93.98 0)
+    (property "Footprint" "Hedgehog:Diode_SOD123" (at 175.26 93.98 0)
       (effects (font (size 1.27 1.27)) hide)
     )
@@
       (effects (font (size 1.27 1.27)) (justify right))
     )
-    (property "Footprint" "Lily58_Pro:Diode_TH_SOD123" (at 195.58 93.98 0)
+    (property "Footprint" "Hedgehog:Diode_SOD123" (at 195.58 93.98 0)
       (effects (font (size 1.27 1.27)) hide)
     )
@@
       (effects (font (size 1.27 1.27)) (justify right))
     )
-    (property "Footprint" "Lily58_Pro:Diode_TH_SOD123" (at 215.9 93.98 0)
+    (property "Footprint" "Hedgehog:Diode_SOD123" (at 215.9 93.98 0)
       (effects (font (size 1.27 1.27)) hide)
     )
@@
       (effects (font (size 1.27 1.27)) (justify right))
     )
-    (property "Footprint" "Lily58_Pro:Diode_TH_SOD123" (at 236.22 93.98 0)
+    (property "Footprint" "Hedgehog:Diode_SOD123" (at 236.22 93.98 0)
       (effects (font (size 1.27 1.27)) hide)
     )
@@
       (effects (font (size 1.27 1.27)) (justify right))
     )
-    (property "Footprint" "Lily58_Pro:Diode_TH_SOD123" (at 256.54 93.98 0)
+    (property "Footprint" "Hedgehog:Diode_SOD123" (at 256.54 93.98 0)
       (effects (font (size 1.27 1.27)) hide)
     )
@@
       (effects (font (size 1.27 1.27)) (justify right))
     )
-    (property "Footprint" "Lily58_Pro:Diode_TH_SOD123" (at 154.94 110.49 0)
+    (property "Footprint" "Hedgehog:Diode_SOD123" (at 154.94 110.49 0)
       (effects (font (size 1.27 1.27)) hide)
     )
@@
       (effects (font (size 1.27 1.27)) (justify right))
     )
-    (property "Footprint" "Lily58_Pro:Diode_TH_SOD123" (at 175.26 110.49 0)
+    (property "Footprint" "Hedgehog:Diode_SOD123" (at 175.26 110.49 0)
       (effects (font (size 1.27 1.27)) hide)
     )
@@
       (effects (font (size 1.27 1.27)) (justify right))
     )
-    (property "Footprint" "Lily58_Pro:Diode_TH_SOD123" (at 195.58 110.49 0)
+    (property "Footprint" "Hedgehog:Diode_SOD123" (at 195.58 110.49 0)
       (effects (font (size 1.27 1.27)) hide)
     )
@@
       (effects (font (size 1.27 1.27)) (justify right))
     )
-    (property "Footprint" "Lily58_Pro:Diode_TH_SOD123" (at 215.9 110.49 0)
+    (property "Footprint" "Hedgehog:Diode_SOD123" (at 215.9 110.49 0)
       (effects (font (size 1.27 1.27)) hide)
     )
@@
       (effects (font (size 1.27 1.27)) (justify right))
     )
-    (property "Footprint" "Lily58_Pro:Diode_TH_SOD123" (at 236.22 110.49 0)
+    (property "Footprint" "Hedgehog:Diode_SOD123" (at 236.22 110.49 0)
       (effects (font (size 1.27 1.27)) hide)
     )
@@
       (effects (font (size 1.27 1.27)) (justify right))
     )
-    (property "Footprint" "Lily58_Pro:Diode_TH_SOD123" (at 256.54 110.49 0)
+    (property "Footprint" "Hedgehog:Diode_SOD123" (at 256.54 110.49 0)
       (effects (font (size 1.27 1.27)) hide)
     )
@@
       (effects (font (size 1.27 1.27)) (justify right))
     )
-    (property "Footprint" "Lily58_Pro:Diode_TH_SOD123" (at 154.94 127 0)
+    (property "Footprint" "Hedgehog:Diode_SOD123" (at 154.94 127 0)
       (effects (font (size 1.27 1.27)) hide)
     )
@@
       (effects (font (size 1.27 1.27)) (justify right))
     )
-    (property "Footprint" "Lily58_Pro:Diode_TH_SOD123" (at 175.26 127 0)
+    (property "Footprint" "Hedgehog:Diode_SOD123" (at 175.26 127 0)
       (effects (font (size 1.27 1.27)) hide)
     )
@@
       (effects (font (size 1.27 1.27)) (justify right))
     )
-    (property "Footprint" "Lily58_Pro:Diode_TH_SOD123" (at 195.58 127 0)
+    (property "Footprint" "Hedgehog:Diode_SOD123" (at 195.58 127 0)
       (effects (font (size 1.27 1.27)) hide)
     )
@@
       (effects (font (size 1.27 1.27)) (justify right))
     )
-    (property "Footprint" "Lily58_Pro:Diode_TH_SOD123" (at 215.9 127 0)
+    (property "Footprint" "Hedgehog:Diode_SOD123" (at 215.9 127 0)
       (effects (font (size 1.27 1.27)) hide)
     )
@@
       (effects (font (size 1.27 1.27)) (justify right))
     )
-    (property "Footprint" "Lily58_Pro:Diode_TH_SOD123" (at 236.22 127 0)
-      (effects (font (size 1.27 1.27)) hide)
-    )
+    (property "Footprint" "Hedgehog:Diode_SOD123" (at 236.22 127 0)
+      (effects (font (size 1.27 1.27)) hide)
+    )
